Commit message: fix a bug in urdf that used a path outside of this project

File: hurba_navigation/urdf/hurba_mecanum.xacro (robot description, xacro)
@@ -65,5 +65,5 @@
       <geometry>
         <!--box size=".4 .4 .4"/-->
-        <mesh filename = "package://hurba_robot/meshes/chassis.dae"/>
+        <mesh filename = "package://hurba_navigation/meshes/chassis.dae"/>
       </geometry>
     </visual>
@@ -113,5 +113,5 @@
       <origin xyz="0.0 0 0" rpy=" 0 1.5708 1.5708"/>
       <geometry>
-        <mesh filename = "package://hurba_robot/meshes/wheel.dae"/>
+        <mesh filename = "package://hurba_navigation/meshes/wheel.dae"/>
         <!--cylinder radius = ".1" length = ".08"/-->
       </geometry>
@@ -138,5 +138,5 @@
       <origin xyz="0 0 0" rpy=" 0 1.5708 1.5708"/>
       <geometry>
-        <mesh filename = "package://hurba_robot/meshes/wheel.dae"/>
+        <mesh filename = "package://hurba_navigation/meshes/wheel.dae"/>
         <!--cylinder radius = ".1" length = ".08"/-->
       </geometry>
@@ -190,5 +190,5 @@
       <origin xyz="0 0 0" rpy=" 0 0 0"/>
       <geometry>
-        <mesh filename = "package://hurba_robot/meshes/hokuyo.dae"/>
+        <mesh filename = "package://hurba_navigation/meshes/hokuyo.dae"/>
       </geometry>
     </visual>
